File: template/project_template.kicad_sch (KiCad schematic)
At the start: 0 parts

Commit message: Initial template setup
Other:
- removed sheet Power - Sequencing
- removed sheet Project Architecture
- added sheet Mechanical (mechanical.kicad_sch)
- note added: "IEC 60062 (European/Precision Style)"
- note added: "Mechanical"
- note removed: "Power - Sequencing"
- note removed: "Project Architecture"
- note removed: "Random Sheet 1"
- note removed: "Random Sheet 2"
- note removed: "Revision History"
- title: Cover Page -> Block Diagram
